Commit message: fixed joint ref axes, rm init pos params, added home pos

File: zeroerr_config/config/zeroerr_arm.ros2_control.xacro (robot description, xacro)
@@ -1,6 +1,5 @@
 <?xml version="1.0"?>
 <robot xmlns:xacro="http://www.ros.org/wiki/xacro">
-    <xacro:macro name="zeroerr_arm_ros2_control" params="name initial_positions_file ros2_control_hardware_type">
-        <xacro:property name="initial_positions" value="${load_yaml(initial_positions_file)['initial_positions']}"/>
+        <xacro:macro name="zeroerr_arm_ros2_control" params="name ros2_control_hardware_type">
         <ros2_control name="${name}" type="system">
             <hardware>
@@ -16,37 +15,25 @@
             <joint name="j1">
                 <command_interface name="position"/>
-                <state_interface name="position">
-                  <param name="initial_value">${initial_positions['j1']}</param>
-                </state_interface>
+                <state_interface name="position"/>
             </joint>
             <joint name="j2">
                 <command_interface name="position"/>
-                <state_interface name="position">
-                  <param name="initial_value">${initial_positions['j2']}</param>
-                </state_interface>
+                <state_interface name="position"/>
             </joint>
             <joint name="j3">
                 <command_interface name="position"/>
-                <state_interface name="position">
-                  <param name="initial_value">${initial_positions['j3']}</param>
-                </state_interface>
+                <state_interface name="position"/>
             </joint>
             <joint name="j4">
                 <command_interface name="position"/>
-                <state_interface name="position">
-                  <param name="initial_value">${initial_positions['j4']}</param>
-                </state_interface>
+                <state_interface name="position"/>
             </joint>
             <joint name="j5">
                 <command_interface name="position"/>
-                <state_interface name="position">
-                  <param name="initial_value">${initial_positions['j5']}</param>
-                </state_interface>
+                <state_interface name="position"/>
             </joint>
             <joint name="j6">
                 <command_interface name="position"/>
-                <state_interface name="position">
-                  <param name="initial_value">${initial_positions['j6']}</param>
-                </state_interface>
+                <state_interface name="position"/>
             </joint>
         </ros2_control>

File: zeroerr_config/config/zeroerr_arm.urdf.xacro (robot description, xacro)
@@ -1,5 +1,4 @@
 <?xml version="1.0"?>
 <robot xmlns:xacro="http://www.ros.org/wiki/xacro" name="zeroerr_arm">
-    <xacro:arg name="initial_positions_file" default="initial_positions.yaml" />
     <xacro:arg name="ros2_control_hardware_type" default="mock_components" />
     <!-- Import zeroerr_arm urdf file -->
@@ -7,4 +6,4 @@
     <!-- Import control_xacro -->
     <xacro:include filename="zeroerr_arm.ros2_control.xacro" />
-    <xacro:zeroerr_arm_ros2_control name="ZeroErrArm" initial_positions_file="$(arg initial_positions_file)" ros2_control_hardware_type="$(arg ros2_control_hardware_type)"/>
+    <xacro:zeroerr_arm_ros2_control name="ZeroErrArm" ros2_control_hardware_type="$(arg ros2_control_hardware_type)"/>
 </robot>

File: zeroerr_description/urdf/zeroerr.urdf (robot description, URDF)
Before this commit: robot zeroerr_arm, 7 links, 6 joints
Joints:
- joint j1: origin xyz=0.0775 -0.0775 0.0389 rpy=1.57 0 0 -> xyz=0.0775 -0.0775 0.0389 rpy=1.57 0 -1.570796327
- joint j2: axis 0 0 1 -> 0 0 -1
- joint j4: axis 0 0 1 -> 0 0 -1
