Commit message: refactor base_link to arm_link, made arm namespace and remapping

File: arm_description/urdf/zeroerr.urdf (robot description, URDF)
Before this commit: robot zeroerr_arm, 7 links, 6 joints
Links:
- removed link base_link
- added link arm_link, mass 0.085937; collision mesh filename=package://arm_description/meshes/arm_link.STL; visual mesh filename=package://arm_description/meshes/arm_link.STL
Joints:
- joint j1: parent base_link -> arm_link

Commit message: modified urdf, added camera link/mesh

File: arm_description/urdf/zeroerr.urdf (robot description, URDF)
Before this commit: robot zeroerr_arm, 7 links, 6 joints
Links:
- removed link arm_link
- added link arm_Link, mass 0.232294593893707; collision mesh filename=package://arm_description/meshes/arm_Link.STL; visual mesh filename=package://arm_description/meshes/arm_Link.STL
- added link camera_Link, mass 0.00120400775794929; collision mesh filename=package://arm_description/meshes/camera_Link.STL; visual mesh filename=package://arm_description/meshes/camera_Link.STL
- link j1_Link: mass 1.13778617636807 -> 1.13778569832606
- link j2_Link: mass 2.70662121520297 -> 2.706624786604
- link j3_Link: mass 1.64557369565779 -> 1.64557213465188
- link j4_Link: mass 0.388500039640416 -> 0.324727718002135
- link j5_Link: mass 0.413553678243016 -> 0.307352171858084
- link j6_Link: mass 0.0395178623740459 -> 0.104910783608116
Joints:
- added joint camera: type fixed, parent j6_Link, child camera_Link, origin xyz=0.073713 -0.0295 -0.0145 rpy=-1.5708 0 1.5708, axis 0 0 0
- joint j1: origin xyz=0.0775 -0.0775 0.0389 rpy=1.57 0 -1.570796327 -> xyz=0.0774999999999998 -0.0775 0.0388999999999997 rpy=1.5707963267949 0 2.51744046366525; parent arm_link -> arm_Link
- joint j2: axis 0 0 -1 -> 0 0 1; origin xyz=0 0.0734000000000014 0 rpy=0 0 0 -> xyz=-0.0491744080889805 0.0734000000000008 0.0354152169144622 rpy=0 0.946644136870351 3.14159265358979
- joint j3: origin xyz=0 0.425 0 rpy=0 0 0 -> xyz=0 -0.425 0 rpy=3.14159265358979 0 0
- joint j4: axis 0 0 -1 -> 0 0 1; origin xyz=0 0.400999999999999 -0.0930934055822586 rpy=0 0 0 -> xyz=0 0.401 0 rpy=3.14159263868863 0 0
- joint j5: origin xyz=0 0.0381316776493207 -0.0379065944177415 rpy=0 0 0 -> xyz=0 -0.0374999756318092 0.0423999994412073 rpy=0 0 0
- joint j6: axis 0 1 0 -> 0 0 1; origin xyz=0 0.0478683223506789 -0.0281658025970178 rpy=-1.5707963267949 0 0 -> xyz=0 -0.0485 0.0375 rpy=3.1416 0 -1.5708

Commit message: added joint limits to urdf, yaml, ec thread prio,

File: arm_description/urdf/zeroerr.urdf (robot description, URDF)
Before this commit: robot ArmProject, 8 links, 7 joints
Joints:
- joint j1: limit (none) -> lower=-3.14 upper=3.14 effort=1000.0 velocity=0.2; type continuous -> revolute
- joint j2: limit (none) -> lower=-3.14 upper=3.14 effort=1000.0 velocity=0.2; type continuous -> revolute
- joint j3: limit (none) -> lower=-3.14 upper=3.14 effort=1000.0 velocity=0.2; type continuous -> revolute
- joint j4: limit (none) -> lower=-3.14 upper=3.14 effort=1000.0 velocity=0.2; type continuous -> revolute
- joint j5: limit (none) -> lower=-3.14 upper=3.14 effort=1000.0 velocity=0.2; type continuous -> revolute
- joint j6: limit (none) -> lower=-3.14 upper=3.14 effort=1000.0 velocity=0.2; type continuous -> revolute
