Commit message: fixed j5/6 in urdf, servo files, launch files

File: arm_description/urdf/zeroerr_cts.urdf (robot description, URDF)
Before this commit: robot ArmProject, 8 links, 7 joints
Joints:
- joint j1: limit lower=-3.14 upper=3.14 effort=1000.0 velocity=0.2 -> (none); type revolute -> continuous
- joint j2: limit lower=-3.14 upper=3.14 effort=1000.0 velocity=0.2 -> (none); type revolute -> continuous
- joint j3: limit lower=-3.14 upper=3.14 effort=1000.0 velocity=0.2 -> (none); type revolute -> continuous
- joint j4: limit lower=-3.14 upper=3.14 effort=1000.0 velocity=0.2 -> (none); type revolute -> continuous
- joint j5: limit lower=-3.14 upper=3.14 effort=1000.0 velocity=0.2 -> (none); type revolute -> continuous
- joint j6: limit lower=-3.14 upper=3.14 effort=1000.0 velocity=0.2 -> (none); type revolute -> continuous
