Commit message: renamed description package, references

File: arm_config/config/zeroerr_arm.ros2_control.xacro (robot description, xacro)
@@ -1,5 +1,5 @@
 <?xml version="1.0"?>
 <robot xmlns:xacro="http://www.ros.org/wiki/xacro">
-        <xacro:macro name="zeroerr_arm_ros2_control" params="name ros2_control_hardware_type">
+        <xacro:macro name="arm_ros2_control" params="name ros2_control_hardware_type">
         <ros2_control name="${name}" type="system">
             <hardware>
@@ -8,5 +8,5 @@
                 </xacro:if>
                 <xacro:if value="${ros2_control_hardware_type == 'real'}">
-                    <plugin>zeroerr_hardware/ArmHardwareInterface</plugin>
+                    <plugin>arm_hardware/ArmHardwareInterface</plugin>
                     <param name="command_interface_topic">arm/command</param>
                     <param name="state_interface_topic">arm/state</param>

File: arm_config/config/zeroerr_arm.urdf.xacro (robot description, xacro)
@@ -3,7 +3,7 @@
     <xacro:arg name="ros2_control_hardware_type" default="mock_components" />
     <!-- Import zeroerr_arm urdf file -->
-    <xacro:include filename="$(find zeroerr_description)/urdf/zeroerr.urdf" />
+    <xacro:include filename="$(find arm_description)/urdf/zeroerr.urdf" />
     <!-- Import control_xacro -->
     <xacro:include filename="zeroerr_arm.ros2_control.xacro" />
-    <xacro:zeroerr_arm_ros2_control name="ZeroErrArm" ros2_control_hardware_type="$(arg ros2_control_hardware_type)"/>
+    <xacro:arm_ros2_control name="ArmProject" ros2_control_hardware_type="$(arg ros2_control_hardware_type)"/>
 </robot>

File: arm_description/urdf/zeroerr.urdf (robot description, URDF)
Before this commit: robot zeroerr_arm, 7 links, 6 joints
Links:
- link base_link: geometry collision mesh filename=package://arm_description/meshes/base_link.STL; visual mesh filename=package://arm_description/meshes/base_link.STL
- link j1_Link: geometry collision mesh filename=package://arm_description/meshes/j1_Link.STL; visual mesh filename=package://arm_description/meshes/j1_Link.STL
- link j2_Link: geometry collision mesh filename=package://arm_description/meshes/j2_Link.STL; visual mesh filename=package://arm_description/meshes/j2_Link.STL
- link j3_Link: geometry collision mesh filename=package://arm_description/meshes/j3_Link.STL; visual mesh filename=package://arm_description/meshes/j3_Link.STL
- link j4_Link: geometry collision mesh filename=package://arm_description/meshes/j4_Link.STL; visual mesh filename=package://arm_description/meshes/j4_Link.STL
- link j5_Link: geometry collision mesh filename=package://arm_description/meshes/j5_Link.STL; visual mesh filename=package://arm_description/meshes/j5_Link.STL
- link j6_Link: geometry collision mesh filename=package://arm_description/meshes/j6_Link.STL; visual mesh filename=package://arm_description/meshes/j6_Link.STL

Commit message: added control mode param, hw interface for manual servo

File: arm_config/config/zeroerr_arm.ros2_control.xacro (robot description, xacro)
@@ -1,5 +1,5 @@
 <?xml version="1.0"?>
 <robot xmlns:xacro="http://www.ros.org/wiki/xacro">
-        <xacro:macro name="arm_ros2_control" params="name ros2_control_hardware_type">
+        <xacro:macro name="arm_ros2_control" params="name ros2_control_hardware_type control_mode">
         <ros2_control name="${name}" type="system">
             <hardware>
@@ -11,4 +11,5 @@
                     <param name="command_interface_topic">arm/command</param>
                     <param name="state_interface_topic">arm/state</param>
+                    <param name="control_mode">${control_mode}</param>
                 </xacro:if>
             </hardware>

File: arm_config/config/zeroerr_arm_servo.urdf.xacro (robot description, xacro)
@@ -1,9 +1,10 @@
 <?xml version="1.0"?>
 <robot xmlns:xacro="http://www.ros.org/wiki/xacro" name="ArmProject">
-    <xacro:arg name="ros2_control_hardware_type" default="mock_components" />
+    <xacro:arg name="ros2_control_hardware_type" default="sim" />
+    <xacro:arg name="control_mode" default="servo" />
     <!-- Import zeroerr_arm urdf file -->
     <xacro:include filename="$(find arm_description)/urdf/zeroerr_cts.urdf" />
     <!-- Import control_xacro -->
     <xacro:include filename="zeroerr_arm.ros2_control.xacro" />
-    <xacro:arm_ros2_control name="ArmProject" ros2_control_hardware_type="$(arg ros2_control_hardware_type)"/>
+    <xacro:arm_ros2_control name="ArmProject" ros2_control_hardware_type="$(arg ros2_control_hardware_type)" control_mode="$(arg control_mode)"/>
 </robot>
